File: pcb-knx-distributor.kicad_sch (KiCad schematic)
At the start: 14 parts, among them J1 Conn_01x02_Pin, J10 Conn_01x02_Pin, J11 Conn_01x02_Pin, J12 Conn_01x02_Pin, J13 Conn_01x02_Pin, J14 Conn_01x02_Pin, J2 Conn_01x02_Pin, J3 Conn_01x02_Pin, J4 Conn_01x02_Pin, J5 Conn_01x02_Pin, J6 Conn_01x02_Pin, J7 Conn_01x02_Pin, J8 Conn_01x02_Pin, J9 Conn_01x02_Pin

Commit message: Updated footprints
Parts:
- J1, J2, J3, J4, J5, J6: footprint haus-automatisierung:Wago-243-131 -> haus-automatisierung:Wago-243-211
- J10, J11, J12, J7, J8, J9: footprint haus-automatisierung:Wago-243-131 -> haus-automatisierung:Wago-243-212
Changed lines of the file:
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@@
     (title "KNX Distributor")
     (date "2023-08-15")
-    (rev "0.1")
+    (rev "0.2")
     (company "haus-automatisierung.com")
     (comment 1 "Matthias Kleine")
@@
       (effects (font (size 1.27 1.27)) (justify right))
     )
-    (property "Footprint" "haus-automatisierung:Wago-243-131" (at 140.335 80.645 0)
+    (property "Footprint" "haus-automatisierung:Wago-243-212" (at 140.335 80.645 0)
       (effects (font (size 1.27 1.27)) hide)
     )
@@
       (effects (font (size 1.27 1.27)) (justify right))
     )
-    (property "Footprint" "haus-automatisierung:Wago-243-131" (at 161.925 80.645 0)
+    (property "Footprint" "haus-automatisierung:Wago-243-212" (at 161.925 80.645 0)
       (effects (font (size 1.27 1.27)) hide)
     )
@@
       (effects (font (size 1.27 1.27)) (justify right))
     )
-    (property "Footprint" "haus-automatisierung:Wago-243-131" (at 52.705 81.28 0)
+    (property "Footprint" "haus-automatisierung:Wago-243-212" (at 52.705 81.28 0)
       (effects (font (size 1.27 1.27)) hide)
     )
@@
       (effects (font (size 1.27 1.27)) (justify right))
     )
-    (property "Footprint" "haus-automatisierung:Wago-243-131" (at 118.11 80.645 0)
+    (property "Footprint" "haus-automatisierung:Wago-243-212" (at 118.11 80.645 0)
       (effects (font (size 1.27 1.27)) hide)
     )
@@
       (effects (font (size 1.27 1.27)) (justify right))
     )
-    (property "Footprint" "haus-automatisierung:Wago-243-131" (at 74.93 80.645 0)
+    (property "Footprint" "haus-automatisierung:Wago-243-212" (at 74.93 80.645 0)
       (effects (font (size 1.27 1.27)) hide)
     )
@@
       (effects (font (size 1.27 1.27)) (justify right))
     )
-    (property "Footprint" "haus-automatisierung:Wago-243-131" (at 74.93 53.975 0)
+    (property "Footprint" "haus-automatisierung:Wago-243-211" (at 74.93 53.975 0)
       (effects (font (size 1.27 1.27)) hide)
     )
@@
       (effects (font (size 1.27 1.27)) (justify right))
     )
-    (property "Footprint" "haus-automatisierung:Wago-243-131" (at 118.11 53.975 0)
+    (property "Footprint" "haus-automatisierung:Wago-243-211" (at 118.11 53.975 0)
       (effects (font (size 1.27 1.27)) hide)
     )
@@
       (effects (font (size 1.27 1.27)) (justify right))
     )
-    (property "Footprint" "haus-automatisierung:Wago-243-131" (at 140.335 53.975 0)
+    (property "Footprint" "haus-automatisierung:Wago-243-211" (at 140.335 53.975 0)
       (effects (font (size 1.27 1.27)) hide)
     )
@@
       (effects (font (size 1.27 1.27)) (justify right))
     )
-    (property "Footprint" "haus-automatisierung:Wago-243-131" (at 52.705 54.61 0)
+    (property "Footprint" "haus-automatisierung:Wago-243-211" (at 52.705 54.61 0)
       (effects (font (size 1.27 1.27)) hide)
     )
@@
       (effects (font (size 1.27 1.27)) (justify right))
     )
-    (property "Footprint" "haus-automatisierung:Wago-243-131" (at 96.52 53.975 0)
+    (property "Footprint" "haus-automatisierung:Wago-243-211" (at 96.52 53.975 0)
       (effects (font (size 1.27 1.27)) hide)
     )
@@
       (effects (font (size 1.27 1.27)) (justify right))
     )
-    (property "Footprint" "haus-automatisierung:Wago-243-131" (at 161.925 53.975 0)
+    (property "Footprint" "haus-automatisierung:Wago-243-211" (at 161.925 53.975 0)
       (effects (font (size 1.27 1.27)) hide)
     )
@@
       (effects (font (size 1.27 1.27)) (justify right))
     )
-    (property "Footprint" "haus-automatisierung:Wago-243-131" (at 96.52 80.645 0)
-      (effects (font (size 1.27 1.27)) hide)
-    )
+    (property "Footprint" "haus-automatisierung:Wago-243-212" (at 96.52 80.645 0)
+      (effects (font (size 1.27 1.27)) hide)
+    )

Commit message: 0.4
Parts:
- added J13: Conn_01x02_Pin, haus-automatisierung:Wago-243-211, symbol Connector:Conn_01x02_Pin
- added J14: Conn_01x02_Pin, haus-automatisierung:Wago-243-212, symbol Connector:Conn_01x02_Pin
- renumbered J11 to J10, J6 to J11, J13 to J15, J14 to J16, J7 to J2, J2 to J3, J8 to J4, J3 to J5, J9 to J6, J4 to J7, J10 to J8, J5 to J9
Connections:
- net black: now also J13.1 (Pin_1)
- net grey: now also J14.1 (Pin_1)
- net red: now also J13.2 (Pin_2)
- net yellow: now also J14.2 (Pin_2)
Other:
- moved on the sheet: J16
