File: pcb-knx-distributor.kicad_pcb (KiCad board)
At the start: 2 copper layers, 107 x 28 mm, 21 parts, among them J1 Conn_01x02_Pin, J10 Conn_01x02_Pin, J11 Conn_01x02_Pin, J12 Conn_01x02_Pin, J13 Conn_01x02_Pin, J14 Conn_01x02_Pin, J15 Conn_01x02_Pin, J16 Conn_01x02_Pin, J2 Conn_01x02_Pin, J3 Conn_01x02_Pin, J4 Conn_01x02_Pin, J5 Conn_01x02_Pin, J6 Conn_01x02_Pin, J7 Conn_01x02_Pin, J8 Conn_01x02_Pin, J9 Conn_01x02_Pin

Commit message: v0.7
Parts:
- removed the G*** at (34.4, 64.0)
- added G***: LOGO, haus-automatisierung:Logo2024-notext, B.Cu at (34.8, 64.0)
- added J17: Conn_01x01_Pin, Connector_PinHeader_2.54mm:PinHeader_1x01_P2.54mm_Vertical, B.Cu at (31.5, 70.0)
- added J18: Conn_01x01_Pin, Connector_PinHeader_2.54mm:PinHeader_1x01_P2.54mm_Vertical, B.Cu at (31.5, 58.0)
- added REF**: WEEE-Logo_5.6x8mm_SilkScreen, Symbol:WEEE-Logo_5.6x8mm_SilkScreen, B.Cu at (117.0, 64.0)
Routing:
- net /black: track 159.3 -> 172.8 mm
- net /red: track 144.9 -> 155.9 mm
Other:
- board text added: "v0.7"
- board text removed: "v0.6"
